Commit message: update

File: core/robot_simulation/urdf/first_robot.urdf (robot description, URDF)
Before this commit: robot first_robot, 2 links, 1 joints
Links:
- link base_link: mass None -> 1.0
- link imu_link: mass None -> 0.001

File: core/robot_simulation/urdf/fishrot/fishbot.xacro (robot description, xacro)
@@ -16,3 +16,18 @@
     <xacro:drive_wheel_xacro wheel_name="right_rear_wheel"   xyz = "-0.25 -0.25 -0.08"/> <!-- 右后驱动轮 -->
     <xacro:caster_wheel_xacro wheel_name="center_caster" xyz = "0 0 -0.096"/> <!-- 中心万向轮 -->
+    <!-- 差速驱动插件（作用在整个模型上） -->
+    <gazebo>
+        <plugin
+            filename="libignition-gazebo-diff-drive-system.so"
+            name="ignition::gazebo::systems::DiffDrive">
+            <left_joint>left_front_wheel_joint</left_joint>
+            <left_joint>left_rear_wheel_joint</left_joint>
+            <right_joint>right_front_wheel_joint</right_joint>
+            <right_joint>right_rear_wheel_joint</right_joint>
+            <wheel_separation>0.5</wheel_separation>
+            <wheel_radius>0.032</wheel_radius>
+            <odom_publish_frequency>30</odom_publish_frequency>
+            <topic>cmd_vel</topic>
+        </plugin>
+    </gazebo>
 </robot>
