Commit message: update

File: core/robot_simulation/urdf/fishrot/base.xacro (robot description, xacro)
@@ -17,4 +17,20 @@
                 </material>
             </visual>
+            <!-- 碰撞体积 (与visual几何一致) -->
+            <collision>
+                <origin xyz="0 0 0" rpy="0 0 0"/>
+                <geometry>
+                    <box size="${length} ${width} ${height}"/>
+                </geometry>
+            </collision>
+            <!-- 惯性 (质量与转动惯量，Gazebo仿真必需) -->
+            <inertial>
+                <mass value="5"/>
+                <!-- 长方体转动惯量: Ixx=m/12*(y²+z²), Iyy=m/12*(x²+z²), Izz=m/12*(x²+y²) -->
+                <inertia ixx="${5.0/12.0 * (width*width + height*height)}"
+                         iyy="${5.0/12.0 * (length*length + height*height)}"
+                         izz="${5.0/12.0 * (length*length + width*width)}"
+                         ixy="0" ixz="0" iyz="0"/>
+            </inertial>
         </link>
     <!-- 添加虚拟部件，使机器人轮子贴合地面 -->

File: core/robot_simulation/urdf/fishrot/caster_wheel.xacro (robot description, xacro)
@@ -16,4 +16,18 @@
                 </material>
             </visual>
+            <!-- 碰撞体积 (与visual几何一致) -->
+            <collision>
+                <origin xyz="0 0 0" rpy="0 0 0"/>
+                <geometry>
+                    <sphere radius="0.016"/>
+                </geometry>
+            </collision>
+            <!-- 惯性 (质量与转动惯量，Gazebo仿真必需) -->
+            <inertial>
+                <mass value="0.05"/>
+                <!-- 球体转动惯量: I = 2/5 * m * r² -->
+                <inertia ixx="0.00000512" iyy="0.00000512" izz="0.00000512"
+                         ixy="0" ixz="0" iyz="0"/>
+            </inertial>
         </link>
         <joint name = "${wheel_name}_joint" type = "fixed">
@@ -22,4 +36,19 @@
             <origin xyz="${xyz}" rpy="0 0 0"/> <!-- child(${${wheel_name}_link) 相对于 parent(base_link) 的偏移 -->
         </joint>
+        <!-- Gazebo Fortress 万向轮接触物理参数，无摩擦可自由滑动 -->
+        <gazebo reference="${wheel_name}_link">
+            <collision>
+                <surface>
+                    <contact>
+                        <ode>
+                            <mu>0.0</mu>      <!-- 滚动摩擦为0，万向轮无阻力 -->
+                            <mu2>0.0</mu2>    <!-- 侧滑摩擦为0，万向轮可自由转向 -->
+                            <kp>10000000000.0</kp> <!-- 接触刚度，避免陷地 -->
+                            <kd>1.0</kd>      <!-- 接触阻尼，落地缓冲 -->
+                        </ode>
+                    </contact>
+                </surface>
+            </collision>
+        </gazebo>
     </xacro:macro>
 </robot>

File: core/robot_simulation/urdf/fishrot/drive_wheel.xacro (robot description, xacro)
@@ -17,4 +17,18 @@
                 </material>
             </visual>
+            <!-- 碰撞体积 (与visual几何一致) -->
+            <collision>
+                <origin xyz="0 0 0" rpy="1.5708 0 0"/>
+                <geometry>
+                    <cylinder radius="0.032" length="0.04"/>
+                </geometry>
+            </collision>
+            <!-- 惯性 (质量与转动惯量，Gazebo仿真必需) -->
+            <inertial>
+                <mass value="0.1"/>
+                <!-- 圆柱体转动惯量 (半径r=0.032, 长l=0.04, 绕轴I=mr²/2, 垂直轴I=m(3r²+l²)/12) -->
+                <inertia ixx="0.0000389" iyy="0.0000512" izz="0.0000389"
+                         ixy="0" ixz="0" iyz="0"/>
+            </inertial>
         </link>
         <joint name = "${wheel_name}_joint" type = "continuous">
@@ -24,4 +38,19 @@
             <axis xyz="0 1 0"/> <!-- 轴向为y轴 -->
         </joint>
+        <!-- Gazebo Fortress 驱动轮接触物理参数，防打滑陷地 -->
+        <gazebo reference="${wheel_name}_link">
+            <collision>
+                <surface>
+                    <contact>
+                        <ode>
+                            <mu>20.0</mu>     <!-- 滚动方向摩擦系数，越大越不打滑 -->
+                            <mu2>20.0</mu2>   <!-- 横向侧滑摩擦系数 -->
+                            <kp>10000000000.0</kp> <!-- 接触刚度，轮子硬度 -->
+                            <kd>1.0</kd>      <!-- 接触阻尼，落地缓冲 -->
+                        </ode>
+                    </contact>
+                </surface>
+            </collision>
+        </gazebo>
     </xacro:macro>
 </robot>

File: core/robot_simulation/urdf/fishrot/imu.xacro (robot description, xacro)
@@ -17,4 +17,17 @@
                 </material>
             </visual>
+            <!-- 碰撞体积 (与visual几何一致) -->
+            <collision>
+                <origin xyz="0 0 0" rpy="0 0 0"/>
+                <geometry>
+                    <box size="0.02 0.02 0.02"/>
+                </geometry>
+            </collision>
+            <!-- 惯性 (质量与转动惯量，Gazebo仿真必需) -->
+            <inertial>
+                <mass value="0.01"/>
+                <inertia ixx="0.000000667" iyy="0.000000667" izz="0.000000667"
+                         ixy="0" ixz="0" iyz="0"/>
+            </inertial>
         </link>
         <!-- 将IMU部件固定到机器人身体部件 -->

File: core/robot_simulation/urdf/fishrot/laser.xacro (robot description, xacro)
@@ -17,4 +17,17 @@
                 </material>
             </visual>
+            <!-- 碰撞体积 (与visual几何一致) -->
+            <collision>
+                <origin xyz="0 0 0" rpy="0 0 0"/>
+                <geometry>
+                    <cylinder radius="0.01" length="0.1"/>
+                </geometry>
+            </collision>
+            <!-- 惯性 (质量与转动惯量，Gazebo仿真必需) -->
+            <inertial>
+                <mass value="0.1"/>
+                <inertia ixx="0.0000858" iyy="0.000005" izz="0.0000858"
+                         ixy="0" ixz="0" iyz="0"/>
+            </inertial>
         </link>
         <!-- 雷达部件 -->
@@ -29,8 +42,21 @@
                 </geometry>
                 <!-- 材质颜色 -->
-                <material name="red">
-                    <color rgba="1 0 0 1.0"/>
+                <material name="black">
+                    <color rgba="0 0 0 1.0"/>
                 </material>
             </visual>
+            <!-- 碰撞体积 (与visual几何一致) -->
+            <collision>
+                <origin xyz="0 0 0" rpy="0 0 0"/>
+                <geometry>
+                    <cylinder radius="0.02" length="0.2"/>
+                </geometry>
+            </collision>
+            <!-- 惯性 (质量与转动惯量，Gazebo仿真必需) -->
+            <inertial>
+                <mass value="0.2"/>
+                <inertia ixx="0.000687" iyy="0.00004" izz="0.000687"
+                         ixy="0" ixz="0" iyz="0"/>
+            </inertial>
         </link>
         <!-- 将雷达固定到支撑杆 -->
@@ -46,4 +72,24 @@
             <origin xyz="${xyz}" rpy="0 0 0"/> <!-- child(laser_cylinder_link) 相对于 parent(base_link) 的偏移 -->
         </joint>
+        <gazebo reference="laser_cylinder_link">
+            <visual>
+                <material>
+                    <ambient>0 0 1 1</ambient>
+                    <diffuse>0 0 1 1</diffuse>
+                    <specular>0.1 0.1 0.1 1</specular>
+                    <emissive>0 0 0 1</emissive>
+                </material>
+            </visual>
+        </gazebo>
+        <gazebo reference="laser_link">
+            <visual>
+                <material>
+                    <ambient>0 0 1 1</ambient>
+                    <diffuse>0 0 1 1</diffuse>
+                    <specular>0.1 0.1 0.1 1</specular>
+                    <emissive>0 0 0 1</emissive>
+                </material>
+            </visual>
+        </gazebo>
     </xacro:macro>
 </robot>

File: install/robot_simulation/share/robot_simulation/urdf/first_robot.xacro (robot description, xacro)
@@ -1,50 +1 @@
-<?xml version="1.0"?>
-<robot xmlns:xacro="http://www.ros.org/wiki/xacro" name = "first_robot">
-    <xacro:macro name = "base_link" params = "length width height">
-        <!-- 机器人的身体部件 -->
-        <link name = "base_link">
-            <!-- 部件的外观描述 -->
-            <visual>
-                <!-- 相对于它所属 link 原点的位置偏移 -->
-                <origin xyz="0 0 0.1" rpy="0 0 0"/>
-                <!-- 几何形状 -->
-                <geometry>
-                    <box size="${length} ${width} ${height}"/>   <!-- 长lengthm 宽widthm 高heightm -->
-                </geometry>
-                <!-- 材质颜色 -->
-                <material name="red">
-                    <color rgba="1 0 0 0.2"/>    <!-- 红 绿 蓝 透明度，范围0~1 -->
-                </material>
-            </visual>
-        </link>
-    </xacro:macro>
-    <xacro:macro name = "imu_link" params = "imu_name xyz">
-        <!-- 机器人的IMU部件 -->
-        <link name = "${imu_name}">
-            <!-- 部件的外观描述 -->
-            <visual>
-                <!-- 相对于它所属 link 原点的位置偏移 -->
-                <origin xyz="0 0 0" rpy="0 0 0"/>
-                <!-- 几何形状 -->
-                <geometry>
-                    <box size="0.02 0.02 0.02"/>   <!-- 长0.02m 宽0.02m 高0.02m -->
-                </geometry>
-                <!-- 材质颜色 -->
-                <material name="gray">
-                    <color rgba="0 0 0 0.5"/>
-                </material>
-            </visual>
-        </link>
-        <!-- 机器人的关节，用于组合机器人的部件 -->
-        <joint name = "${imu_name}_joint" type = "fixed">
-            <parent link = "base_link"/>
-            <child link = "${imu_name}"/>
-            <origin xyz="${xyz}" rpy="0 0 0"/> <!-- child(${imu_name}) 相对于 parent(base_link) 的偏移 -->
-        </joint>
-    </xacro:macro>
-    <!-- 机器人的身体部件 -->
-    <xacro:base_link length="0.5" width="0.3" height="0.1"/>
-    <!-- 机器人的IMU部件 -->
-    <xacro:imu_link imu_name="imu_up" xyz="0 0 0.03"/>
-    <xacro:imu_link imu_name="imu_down" xyz="0 0 -0.03"/>
-</robot>
+/home/jinyicheng/auto_navigation/core/robot_simulation/urdf/first_robot.xacro

File: install/robot_simulation/share/robot_simulation/urdf/fishrot/base.xacro (robot description, xacro)
@@ -1,28 +1 @@
-<?xml version="1.0"?>
-<robot xmlns:xacro="http://www.ros.org/wiki/xacro">
-    <xacro:macro name = "base_xacro" params = "length width height">
-        <!-- 机器人的身体部件 -->
-        <link name = "base_link">
-            <!-- 部件的外观描述 -->
-            <visual>
-                <!-- 相对于它所属 link 原点的位置偏移 -->
-                <origin xyz="0 0 0" rpy="0 0 0"/>
-                <!-- 几何形状 -->
-                <geometry>
-                    <box size="${length} ${width} ${height}"/>   <!-- 长lengthm 宽widthm 高heightm -->
-                </geometry>
-                <!-- 材质颜色 -->
-                <material name="red">
-                    <color rgba="1 0 0 0.2"/>    <!-- 红 绿 蓝 透明度，范围0~1 -->
-                </material>
-            </visual>
-        </link>
-    <!-- 添加虚拟部件，使机器人轮子贴合地面 -->
-    <link name = "base_footprint"/>
-    <joint name = "base_footprint_joint" type = "fixed">
-        <parent link = "base_footprint"/>
-        <child link = "base_link"/>
-        <origin xyz="0 0 0.112" rpy="0 0 0"/> <!-- base_link 在 base_footprint 上方 0.112m，轮子恰好贴地 -->
-    </joint>
-    </xacro:macro>
-</robot>
+/home/jinyicheng/auto_navigation/core/robot_simulation/urdf/fishrot/base.xacro

File: install/robot_simulation/share/robot_simulation/urdf/fishrot/caster_wheel.xacro (robot description, xacro)
@@ -1,25 +1 @@
-<?xml version="1.0"?>
-<robot xmlns:xacro="http://www.ros.org/wiki/xacro">
-    <xacro:macro name = "caster_wheel_xacro" params = "wheel_name xyz">
-        <link name = "${wheel_name}_link">
-            <!-- 部件的外观描述 -->
-            <visual>
-                <!-- 相对于它所属 link 原点的位置偏移 -->
-                <origin xyz="0 0 0" rpy="0 0 0"/>
-                <!-- 几何形状 -->
-                <geometry>
-                    <sphere radius="0.016"/>   <!-- 半径0.016m -->
-                </geometry>
-                <!-- 材质颜色 -->
-                <material name="yellow">
-                    <color rgba="1 1 0 0.8"/>    <!-- 红 绿 蓝 透明度，范围0~1 -->
-                </material>
-            </visual>
-        </link>
-        <joint name = "${wheel_name}_joint" type = "fixed">
-            <parent link = "base_link"/>
-            <child link = "${wheel_name}_link"/>
-            <origin xyz="${xyz}" rpy="0 0 0"/> <!-- child(${${wheel_name}_link) 相对于 parent(base_link) 的偏移 -->
-        </joint>
-    </xacro:macro>
-</robot>
+/home/jinyicheng/auto_navigation/core/robot_simulation/urdf/fishrot/caster_wheel.xacro

File: install/robot_simulation/share/robot_simulation/urdf/fishrot/drive_wheel.xacro (robot description, xacro)
@@ -1,27 +1 @@
-<?xml version="1.0"?>
-<robot xmlns:xacro="http://www.ros.org/wiki/xacro">
-    <xacro:macro name = "drive_wheel_xacro" params = "wheel_name xyz">
-        <link name = "${wheel_name}_link">
-            <!-- 部件的外观描述 -->
-            <visual>
-                <!-- 相对于它所属 link 原点的位置偏移 -->
-                <!-- 1.5708弧度，表示绕X轴旋转90度，把竖直的圆柱体放平成轮子 -->
-                <origin xyz="0 0 0" rpy="1.5708 0 0"/>
-                <!-- 几何形状 -->
-                <geometry>
-                    <cylinder radius="0.032" length="0.04"/>   <!-- 半径0.032m 高0.04m -->
-                </geometry>
-                <!-- 材质颜色 -->
-                <material name="yellow">
-                    <color rgba="1 1 0 0.8"/>    <!-- 红 绿 蓝 透明度，范围0~1 -->
-                </material>
-            </visual>
-        </link>
-        <joint name = "${wheel_name}_joint" type = "continuous">
-            <parent link = "base_link"/>
-            <child link = "${wheel_name}_link"/>
-            <origin xyz="${xyz}" rpy="0 0 0"/> <!-- child(${${wheel_name}_link) 相对于 parent(base_link) 的偏移 -->
-            <axis xyz="0 1 0"/> <!-- 轴向为y轴 -->
-        </joint>
-    </xacro:macro>
-</robot>
+/home/jinyicheng/auto_navigation/core/robot_simulation/urdf/fishrot/drive_wheel.xacro

File: install/robot_simulation/share/robot_simulation/urdf/fishrot/fishbot.xacro (robot description, xacro)
@@ -1,18 +1 @@
-<?xml version="1.0"?>
-<robot name="fishbot" xmlns:xacro="http://www.ros.org/wiki/xacro">
-    <!-- 包含机器人的身体部件 -->
-    <xacro:include filename="base.xacro"/>
-    <xacro:include filename="imu.xacro"/>
-    <xacro:include filename="laser.xacro"/>
-    <xacro:include filename="drive_wheel.xacro"/>
-    <xacro:include filename="caster_wheel.xacro"/>
-    <!-- 调用宏 -->
-    <xacro:base_xacro length="0.5" width="0.5" height="0.1"/> <!-- 机器人的身体部件 -->
-    <xacro:imu_xacro xyz = "0 0 -0.1"/> <!-- 机器人的IMU部件 -->
-    <xacro:laser_xacro xyz = "0 0 0.1"/> <!-- 机器人的激光雷达部件 -->
-    <xacro:drive_wheel_xacro wheel_name="left_front_wheel"   xyz = " 0.25  0.25 -0.08"/> <!-- 左前驱动轮 -->
-    <xacro:drive_wheel_xacro wheel_name="right_front_wheel"  xyz = " 0.25 -0.25 -0.08"/> <!-- 右前驱动轮 -->
-    <xacro:drive_wheel_xacro wheel_name="left_rear_wheel"    xyz = "-0.25  0.25 -0.08"/> <!-- 左后驱动轮 -->
-    <xacro:drive_wheel_xacro wheel_name="right_rear_wheel"   xyz = "-0.25 -0.25 -0.08"/> <!-- 右后驱动轮 -->
-    <xacro:caster_wheel_xacro wheel_name="center_caster" xyz = "0 0 -0.096"/> <!-- 中心万向轮 -->
-</robot>
+/home/jinyicheng/auto_navigation/core/robot_simulation/urdf/fishrot/fishbot.xacro

File: install/robot_simulation/share/robot_simulation/urdf/fishrot/imu.xacro (robot description, xacro)
@@ -1,27 +1 @@
-<?xml version="1.0"?>
-<robot xmlns:xacro="http://www.ros.org/wiki/xacro">
-    <xacro:macro name = "imu_xacro" params = "xyz">
-        <!-- 机器人的IMU部件 -->
-        <link name = "imu_link">
-            <!-- 部件的外观描述 -->
-            <visual>
-                <!-- 相对于它所属 link 原点的位置偏移 -->
-                <origin xyz="0 0 0" rpy="0 0 0"/>
-                <!-- 几何形状 -->
-                <geometry>
-                    <box size="0.02 0.02 0.02"/>   <!-- 长0.02m 宽0.02m 高0.02m -->
-                </geometry>
-                <!-- 材质颜色 -->
-                <material name="gray">
-                    <color rgba="0 0 0 0.5"/>
-                </material>
-            </visual>
-        </link>
-        <!-- 将IMU部件固定到机器人身体部件 -->
-        <joint name = "imu_link_joint" type = "fixed">
-            <parent link = "base_link"/>
-            <child link = "imu_link"/>
-            <origin xyz="${xyz}" rpy="0 0 0"/> <!-- child(imu_link) 相对于 parent(base_link) 的偏移 -->
-        </joint>
-    </xacro:macro>
-</robot>
+/home/jinyicheng/auto_navigation/core/robot_simulation/urdf/fishrot/imu.xacro

File: install/robot_simulation/share/robot_simulation/urdf/fishrot/laser.xacro (robot description, xacro)
@@ -1,49 +1 @@
-<?xml version="1.0"?>
-<robot xmlns:xacro="http://www.ros.org/wiki/xacro">
-    <xacro:macro name = "laser_xacro" params = "xyz">
-        <!-- 雷达支撑杆部件 -->
-        <link name = "laser_cylinder_link">
-            <!-- 部件的外观描述 -->
-            <visual>
-                <!-- 相对于它所属 link 原点的位置偏移 -->
-                <origin xyz="0 0 0" rpy="0 0 0"/>
-                <!-- 几何形状 -->
-                <geometry>
-                    <cylinder radius = "0.01" length = "0.1"/>  <!-- 圆柱体：半径0.01m 高0.1m -->
-                </geometry>
-                <!-- 材质颜色 -->
-                <material name="black">
-                    <color rgba="0 0 0 1.0"/>
-                </material>
-            </visual>
-        </link>
-        <!-- 雷达部件 -->
-        <link name = "laser_link">
-            <!-- 部件的外观描述 -->
-            <visual>
-                <!-- 相对于它所属 link 原点的位置偏移 -->
-                <origin xyz="0 0 0" rpy="0 0 0"/>
-                <!-- 几何形状 -->
-                <geometry>
-                    <cylinder radius = "0.02" length = "0.2"/>  <!-- 圆柱体：半径0.02m 高0.2m -->
-                </geometry>
-                <!-- 材质颜色 -->
-                <material name="red">
-                    <color rgba="1 0 0 1.0"/>
-                </material>
-            </visual>
-        </link>
-        <!-- 将雷达固定到支撑杆 -->
-        <joint name = "laser_joint" type = "fixed">
-            <parent link = "laser_cylinder_link"/>
-            <child link = "laser_link"/>
-            <origin xyz="0 0 0.05" rpy="0 0 0"/> <!-- child(laser_link) 相对于 parent(laser_cylinder_link) 的偏移 -->
-        </joint>
-        <!-- 将雷达支撑杆固定到机器人身体 -->
-        <joint name = "laser_cylinder_joint" type = "fixed">
-            <parent link = "base_link"/>
-            <child link = "laser_cylinder_link"/>
-            <origin xyz="${xyz}" rpy="0 0 0"/> <!-- child(laser_cylinder_link) 相对于 parent(base_link) 的偏移 -->
-        </joint>
-    </xacro:macro>
-</robot>
+/home/jinyicheng/auto_navigation/core/robot_simulation/urdf/fishrot/laser.xacro
